File: Module Current Probe.sch (EAGLE design)
At the start: 9 parts, among them J1 CON_HEADER_2X08-PTH-SHROUDED, J2 CON_HEADER_2X08-PTH-SHROUDED, J3 BANANA-JACK, J4 BANANA-JACK, J5 BANANA-JACK, J6 BANANA-JACK, J7 BANANA-JACK, J8 BANANA-JACK

Commit message: Added ground connection for connecting a lab power supply.
Parts:
- added J9: BANANA-JACK, con-banana:BANANA-JACK
Connections:
- net GND: now also J9.PIN
Changed lines of the file:
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@@
 <part name="JP1" library="pinhead" deviceset="PINHD-2X8" device=""/>
 <part name="FRAME1" library="frames" deviceset="DINA4_L" device=""/>
+<part name="J9" library="con-banana" deviceset="BANANA-JACK" device=""/>
 </parts>
 <sheets>
@@
 <attribute name="SHEET" x="248.92" y="1.27" size="2.54" layer="94" font="vector"/>
 </instance>
+<instance part="J9" gate="G$1" x="129.54" y="137.16" rot="R180"/>
 </instances>
 <busses>
@@
 <pinref part="JP1" gate="A" pin="7"/>
 </segment>
+<segment>
+<pinref part="J9" gate="G$1" pin="PIN"/>
+<wire x1="127" y1="137.16" x2="116.84" y2="137.16" width="0.1524" layer="91"/>
+<label x="116.84" y="137.16" size="1.778" layer="95"/>
+</segment>
 </net>
